File: Shematic/board_schematic.sch (EAGLE design)
At the start: 21 parts, among them IC1 MEGA8-P, IC2 L293D, IC3 L293D

Commit message: added some outputs
Parts:
- removed C6: 100nF, rcl:C-EU050-045X075
- added BATTERY_VOLTAGE, SENSOR_0_DATA, SENSOR_1_DATA, SENSOR_2_DATA, TRIG_SENSOR_0, TRIG_SENSOR_1, TRIG_SENSOR_2: WIREPAD2,54/1,0, wirepad:WIREPAD2,54/1,0
- added C7, C8, C9: 470uF, resistor:CPOL-EUE3.5-8
- added I2C, JP5, JP6, JP7: (no value), pinhead:PINHD-1X2
- added LED1, LED2: (no value), led:LED5MM
- added PAD8: WIREPAD2,54/0,9, wirepad:WIREPAD2,54/0,9
- added R1, R3, R5: 1k, eagle-ltspice:R0204/7
- added R2, R4, R6: 81, eagle-ltspice:R0204/7
- added R7: 2.2k, eagle-ltspice:R0204/7
- added R8, R9: 2.7k, eagle-ltspice:R0204/7
- added SERWO: (no value), pinhead:PINHD-2X3
- added T1, T2, T3: (no value), transistor-neu-to92:2N2222-NPN-TO92-EBC
- renumbered PAD1 to MOTOR_2_1, PAD2 to MOTOR_2_2, PAD3 to MOTOR_1_1, PAD4 to MOTOR_1_2
Connections:
- removed net N$16: IC1.PC4(ADC4/SDA), JP1.5
- removed net N$27: IC1.PD7(AIN1), JP3.3
- new net BLABLA: I2C.1, IC1.PC4(ADC4/SDA), JP1.5
- new net N$29: R2.1, T1.C
- new net N$30: R2.2, TRIG_SENSOR_0.P
- new net N$32: R3.2, T2.B
- new net N$33: R4.1, T2.C
- new net N$34: R4.2, TRIG_SENSOR_1.P
- new net N$36: R5.2, T3.B
- new net N$37: R6.1, T3.C
- new net N$38: R6.2, TRIG_SENSOR_2.P
- new net N$5: R1.2, T1.B
- new net PB4: IC1.PB4(MISO), JP2.4, SERWO.1
- new net PD5: IC1.PD5(T1), JP3.1, R1.1
- new net PD6: IC1.PD6(AIN0), JP3.2, R3.1
- new net PD7: IC1.PD7(AIN1), JP3.3, R5.1
- net GND: now also C7.-, C8.-, C9.-, JP7.1, JP7.2, LED1.C, LED2.C, PAD8.P, SERWO.5, T1.E, T2.E, T3.E; no longer C6.1
- net LOGIC_VCC: now also C7.+, C8.+, JP6.1, JP6.2, R8.2, R9.2, SERWO.2
- net N$13: now also SENSOR_1_DATA.P
- net N$14: now also SENSOR_2_DATA.P
- net N$15: now also BATTERY_VOLTAGE.P
- net N$17: now also I2C.2
- net N$18: now also LED1.A, R7.1; no longer IC1.PB4(MISO), JP2.4
- net N$25: now also SERWO.3, SERWO.4; no longer IC1.PD5(T1), JP3.1
- net N$26: now also LED2.A, R8.1; no longer IC1.PD6(AIN0), JP3.2
- net N$9: now also SENSOR_0_DATA.P
- net RESET: now also IC1.PC6(/RESET), R9.1
- net VCC: now also C9.+, JP5.1, JP5.2, R7.2, SERWO.6
Other:
- moved on the sheet: C1, C2, JP1, PAD5, PAD6, PAD7
